Commit message: update readme

File: app/src/hiwonder_xarm_esp32_description/urdf/hiwonder_esp32_gripper.xacro (robot description, xacro)
@@ -2,8 +2,10 @@
 <robot xmlns:xacro="http://www.ros.org/wiki/xacro">
   <!-- ==================== GRIPPER (prismatic simplification) ==================== -->
-  <!-- Tool centre point: measured centre between the two gripping fingers. -->
+  <!-- Tool centre point: estimated centre of a 40 mm ball held between the fingers.
+       Image measurement: 10.5 cm from wrist; ruler check: about 11 cm (2026-10-01).
+       This grasp reference still needs physical validation. -->
   <link name="gripper_tcp_link"/>
   <joint name="gripper_tcp_joint" type="fixed">
-    <origin xyz="0.0 -0.08 0.0" rpy="0.0 0.0 0.0"/>
+    <origin xyz="0.0207 -0.1025 -0.0068" rpy="0.0 0.0 0.0"/>
     <parent link="limb5_link"/>
     <child link="gripper_tcp_link"/>

File: app/src/hiwonder_xarm_esp32_moveit_config/config/hiwonder_esp32.ros2_control.xacro (robot description, xacro)
@@ -126,4 +126,6 @@
         <param name="raw_max">786</param>
         <param name="movement_duration_ms">1000</param>
+        <!-- Slow closure only; opening and arm movements keep their durations. -->
+        <param name="closing_movement_duration_ms">3000</param>
         <param name="hardware_io_enabled">${gripper_hardware_io_enabled}</param>
         <command_interface name="position">
