Commit message: moveit and real physique connection

File: app/src/hiwonder_xarm_esp32_description/urdf/hiwonder_esp32_arm.xacro (robot description, xacro)
@@ -47,6 +47,6 @@
     <parent link="base_link"/>
     <child link="limb1_link"/>
-    <axis xyz="0.0 0.0 -1.0"/>
-    <limit lower="-2.793" upper="2.793" effort="10" velocity="2.0"/>
+    <axis xyz="0.0 0.0 1.0"/>
+    <limit lower="-1.999726" upper="2.021513" effort="10" velocity="2.0"/>
   </joint>
   <link name="limb2_link">
@@ -129,5 +129,5 @@
     <child link="limb4_link"/>
     <axis xyz="-1.0 0.0012 0.0002"/>
-    <limit lower="-2.094" upper="2.094" effort="17" velocity="2.7"/>
+    <limit lower="-1.780316" upper="1.558151" effort="17" velocity="2.7"/>
   </joint>
   <!-- ==================== WRIST (limb5 = gripper base) ==================== -->
@@ -156,6 +156,6 @@
     <parent link="limb4_link"/>
     <child link="limb5_link"/>
-    <axis xyz="0.0 1.0 0.0"/>
-    <limit lower="-1.571" upper="1.571" effort="25" velocity="2.6"/>
+    <axis xyz="0.0 -1.0 0.0"/>
+    <limit lower="-1.562524" upper="1.365440" effort="25" velocity="2.6"/>
   </joint>
 </robot>

File: app/src/hiwonder_xarm_esp32_description/urdf/hiwonder_esp32_gripper.xacro (robot description, xacro)
@@ -2,4 +2,11 @@
 <robot xmlns:xacro="http://www.ros.org/wiki/xacro">
   <!-- ==================== GRIPPER (prismatic simplification) ==================== -->
+  <!-- Tool centre point: measured centre between the two gripping fingers. -->
+  <link name="gripper_tcp_link"/>
+  <joint name="gripper_tcp_joint" type="fixed">
+    <origin xyz="0.0 -0.08 0.0" rpy="0.0 0.0 0.0"/>
+    <parent link="limb5_link"/>
+    <child link="gripper_tcp_link"/>
+  </joint>
   <!-- Gears, fixed visual elements -->
   <link name="gear_left_link">
@@ -79,5 +86,5 @@
     <child link="gripper_left_link"/>
     <axis xyz="1.0 0.0 0.0"/>
-    <limit lower="-0.015" upper="0.015" effort="10" velocity="0.1"/>
+    <limit lower="-0.013921" upper="0.013921" effort="10" velocity="0.1"/>
   </joint>
   <!-- Right finger, mimic left -->
@@ -107,5 +114,5 @@
     <child link="gripper_right_link"/>
     <axis xyz="1.0 0.0 0.0"/>
-    <limit lower="-0.015" upper="0.015" effort="10" velocity="0.1"/>
+    <limit lower="-0.013921" upper="0.013921" effort="10" velocity="0.1"/>
     <mimic joint="gripper_left_joint" multiplier="-1" offset="0"/>
   </joint>

File: app/src/hiwonder_xarm_esp32_moveit_config/config/hiwonder_esp32.ros2_control.xacro (robot description, xacro)
@@ -3,10 +3,10 @@
   <xacro:macro
     name="hiwonder_esp32_ros2_control"
-    params="name initial_positions_file use_mock_hardware serial_port gripper_hardware_io_enabled:=false read_only:=false">
+    params="name initial_positions_file use_mock_hardware serial_port gripper_hardware_io_enabled:=true read_only:=false">
     <xacro:property
       name="initial_positions"
       value="${xacro.load_yaml(initial_positions_file)['initial_positions']}"/>
     <xacro:property name="radians_per_raw" value="${4.1887902047863905 / 1000.0}"/>
-    <xacro:property name="gripper_units_per_raw" value="${0.03 / 540.0}"/>
+    <xacro:property name="gripper_units_per_raw" value="${0.03 / 556.0}"/>
     <ros2_control name="${name}" type="system">
       <hardware>
@@ -26,8 +26,5 @@
         </xacro:unless>
       </hardware>
-      <!--
-        direction=+1 is provisional.  The raw ranges below are measured safe ranges;
-        the ROS direction still needs joint-by-joint RViz validation before motion.
-      -->
+      <!-- Raw ranges include a 20-unit margin from the measured positions. -->
       <joint name="limb1_to_base_link_joint">
         <param name="servo_id">6</param>
@@ -35,11 +32,11 @@
         <param name="ros_reference">0.015082</param>
         <param name="units_per_raw">${radians_per_raw}</param>
-        <param name="direction">-1</param>
+        <param name="direction">1</param>
         <param name="raw_min">20</param>
         <param name="raw_max">980</param>
         <param name="hardware_io_enabled">true</param>
         <command_interface name="position">
-          <param name="min">-1.99135</param>
-          <param name="max">2.02989</param>
+          <param name="min">-1.999726</param>
+          <param name="max">2.021513</param>
         </command_interface>
         <state_interface name="position">
@@ -86,14 +83,14 @@
       <joint name="limb4_to_limb3_joint">
         <param name="servo_id">3</param>
-        <param name="raw_reference">127</param>
-        <param name="ros_reference">-1.573432</param>
+        <param name="raw_reference">503</param>
+        <param name="ros_reference">0.071130</param>
         <param name="units_per_raw">${radians_per_raw}</param>
         <param name="direction">1</param>
-        <param name="raw_min">69</param>
-        <param name="raw_max">980</param>
+        <param name="raw_min">61</param>
+        <param name="raw_max">858</param>
         <param name="hardware_io_enabled">true</param>
         <command_interface name="position">
-          <param name="min">-1.81638</param>
-          <param name="max">1.99961</param>
+          <param name="min">-1.780316</param>
+          <param name="max">1.558151</param>
         </command_interface>
         <state_interface name="position">
@@ -107,11 +104,11 @@
         <param name="ros_reference">-0.008483</param>
         <param name="units_per_raw">${radians_per_raw}</param>
-        <param name="direction">-1</param>
-        <param name="raw_min">26</param>
-        <param name="raw_max">959</param>
+        <param name="direction">1</param>
+        <param name="raw_min">141</param>
+        <param name="raw_max">840</param>
         <param name="hardware_io_enabled">true</param>
         <command_interface name="position">
-          <param name="min">-1.88087</param>
-          <param name="max">2.02727</param>
+          <param name="min">-1.562524</param>
+          <param name="max">1.365440</param>
         </command_interface>
         <state_interface name="position">
@@ -122,20 +119,15 @@
       <joint name="gripper_left_joint">
         <param name="servo_id">1</param>
-        <param name="raw_reference">443</param>
+        <param name="raw_reference">528</param>
         <param name="ros_reference">0.0</param>
         <param name="units_per_raw">${gripper_units_per_raw}</param>
-        <param name="direction">1</param>
-        <!--
-          Servo 1 cable is broken.  Expose a fixed state and never address this
-          servo unless this per-joint parameter is deliberately enabled again.
-          Its ROS direction/gripper geometry has not been validated, so its ROS
-          command limits remain unchanged despite the updated raw range.
-        -->
-        <param name="raw_min">100</param>
-        <param name="raw_max">647</param>
+        <param name="direction">-1</param>
+        <param name="raw_min">270</param>
+        <param name="raw_max">786</param>
+        <param name="movement_duration_ms">1000</param>
         <param name="hardware_io_enabled">${gripper_hardware_io_enabled}</param>
         <command_interface name="position">
-          <param name="min">-0.015</param>
-          <param name="max">0.0112222</param>
+          <param name="min">-0.013921</param>
+          <param name="max">0.013921</param>
         </command_interface>
         <state_interface name="position">

File: app/src/hiwonder_xarm_esp32_moveit_config/config/hiwonder_esp32.urdf.xacro (robot description, xacro)
@@ -4,6 +4,5 @@
     <xacro:arg name="use_mock_hardware" default="true" />
     <xacro:arg name="serial_port" default="/dev/ttyUSB0" />
-    <!-- Keep ID 1 isolated until its broken cable has been repaired and revalidated. -->
-    <xacro:arg name="gripper_hardware_io_enabled" default="false" />
+    <xacro:arg name="gripper_hardware_io_enabled" default="true" />
     <xacro:arg name="read_only" default="false" />
     <!-- Import hiwonder_esp32 urdf file -->

Commit message: Fix the tilted desk with calibrated servo scales and joint limits, and make ball picking more robust.

File: app/src/hiwonder_xarm_esp32_description/urdf/hiwonder_esp32_arm.xacro (robot description, xacro)
@@ -48,5 +48,5 @@
     <child link="limb1_link"/>
     <axis xyz="0.0 0.0 1.0"/>
-    <limit lower="-1.999726" upper="2.021513" effort="10" velocity="2.0"/>
+    <limit lower="-2.020670" upper="2.042456" effort="10" velocity="2.0"/>
   </joint>
   <link name="limb2_link">
@@ -129,5 +129,5 @@
     <child link="limb4_link"/>
     <axis xyz="-1.0 0.0012 0.0002"/>
-    <limit lower="-1.780316" upper="1.558151" effort="17" velocity="2.7"/>
+    <limit lower="-1.885517" upper="1.646953" effort="17" velocity="2.7"/>
   </joint>
   <!-- ==================== WRIST (limb5 = gripper base) ==================== -->
@@ -157,5 +157,5 @@
     <child link="limb5_link"/>
     <axis xyz="0.0 -1.0 0.0"/>
-    <limit lower="-1.562524" upper="1.365440" effort="25" velocity="2.6"/>
+    <limit lower="-1.583468" upper="1.386384" effort="25" velocity="2.6"/>
   </joint>
 </robot>

File: app/src/hiwonder_xarm_esp32_moveit_config/config/hiwonder_esp32.ros2_control.xacro (robot description, xacro)
@@ -8,4 +8,10 @@
       value="${xacro.load_yaml(initial_positions_file)['initial_positions']}"/>
     <xacro:property name="radians_per_raw" value="${4.1887902047863905 / 1000.0}"/>
+    <!-- Servos turn more than the nominal 240 deg per 1000 raw units. Scales measured
+         on 2026-10-16 by moving one joint and measuring the camera rotation on a fixed
+         checkerboard. The base and wrist rotation keep the nominal value. -->
+    <xacro:property name="shoulder_radians_per_raw" value="${radians_per_raw * 1.070}"/>
+    <xacro:property name="elbow_radians_per_raw" value="${radians_per_raw * 1.056}"/>
+    <xacro:property name="wrist_radians_per_raw" value="${radians_per_raw * 1.045}"/>
     <xacro:property name="gripper_units_per_raw" value="${0.03 / 556.0}"/>
     <ros2_control name="${name}" type="system">
@@ -22,9 +28,14 @@
           <param name="startup_delay_ms">2000</param>
           <param name="movement_duration_ms">40</param>
+          <!-- A lost servo reply keeps the last position for up to 5 cycles. -->
+          <param name="max_consecutive_read_failures">5</param>
           <!-- read_only suppresses every hardware output in HiwonderSystem. -->
           <param name="read_only">${read_only}</param>
         </xacro:unless>
       </hardware>
-      <!-- Raw ranges include a 20-unit margin from the measured positions. -->
+      <!-- Raw ranges include a 20-unit margin from the measured positions. The plugin
+           clamps commands to them. The min and max below extend them by 5 raw units so
+           a servo settling just past its commanded limit does not stop the controllers;
+           MoveIt plans 10 units inside them (joint_limits.yaml). -->
       <joint name="limb1_to_base_link_joint">
         <param name="servo_id">6</param>
@@ -37,6 +48,6 @@
         <param name="hardware_io_enabled">true</param>
         <command_interface name="position">
-          <param name="min">-1.999726</param>
-          <param name="max">2.021513</param>
+          <param name="min">-2.020670</param>
+          <param name="max">2.042456</param>
         </command_interface>
         <state_interface name="position">
@@ -49,5 +60,5 @@
         <param name="raw_reference">856</param>
         <param name="ros_reference">1.550816</param>
-        <param name="units_per_raw">${radians_per_raw}</param>
+        <param name="units_per_raw">${shoulder_radians_per_raw}</param>
         <param name="direction">1</param>
         <param name="raw_min">119</param>
@@ -55,6 +66,6 @@
         <param name="hardware_io_enabled">true</param>
         <command_interface name="position">
-          <param name="min">-1.53632</param>
-          <param name="max">1.52149</param>
+          <param name="min">-1.774832</param>
+          <param name="max">1.541852</param>
         </command_interface>
         <state_interface name="position">
@@ -67,5 +78,5 @@
         <param name="raw_reference">863</param>
         <param name="ros_reference">1.550816</param>
-        <param name="units_per_raw">${radians_per_raw}</param>
+        <param name="units_per_raw">${elbow_radians_per_raw}</param>
         <param name="direction">1</param>
         <param name="raw_min">20</param>
@@ -73,6 +84,6 @@
         <param name="hardware_io_enabled">true</param>
         <command_interface name="position">
-          <param name="min">-1.98033</param>
-          <param name="max">2.04090</param>
+          <param name="min">-2.094</param>
+          <param name="max">2.090466</param>
         </command_interface>
         <state_interface name="position">
@@ -85,5 +96,5 @@
         <param name="raw_reference">503</param>
         <param name="ros_reference">0.071130</param>
-        <param name="units_per_raw">${radians_per_raw}</param>
+        <param name="units_per_raw">${wrist_radians_per_raw}</param>
         <param name="direction">1</param>
         <param name="raw_min">61</param>
@@ -91,6 +102,6 @@
         <param name="hardware_io_enabled">true</param>
         <command_interface name="position">
-          <param name="min">-1.780316</param>
-          <param name="max">1.558151</param>
+          <param name="min">-1.885517</param>
+          <param name="max">1.646953</param>
         </command_interface>
         <state_interface name="position">
@@ -109,6 +120,6 @@
         <param name="hardware_io_enabled">true</param>
         <command_interface name="position">
-          <param name="min">-1.562524</param>
-          <param name="max">1.365440</param>
+          <param name="min">-1.583468</param>
+          <param name="max">1.386384</param>
         </command_interface>
         <state_interface name="position">
@@ -126,6 +137,6 @@
         <param name="raw_max">786</param>
         <param name="movement_duration_ms">1000</param>
-        <!-- Slow closure only; opening and arm movements keep their durations. -->
-        <param name="closing_movement_duration_ms">3000</param>
+        <!-- Closing duration is independent of opening and arm movements. -->
+        <param name="closing_movement_duration_ms">500</param>
         <param name="hardware_io_enabled">${gripper_hardware_io_enabled}</param>
         <command_interface name="position">
